File: lt_SOM_socket.sch (KiCad schematic (older format))
At the start: 0 parts

Commit message: SOM added.
Signed-off-by: Kali Prasad <kprasadvnsi@protonmail.com>
Parts:
- added J? (x2): Conn_01x40_Female, symbol Connector:Conn_01x40_Female
Connections:
- new net +3V3: J?.5 (Pin_5)
- new net +5V: J?.3 (Pin_3)
- new net A11: J?.16 (Pin_16)
- new net A12: J?.20 (Pin_20)
- new net A13: J?.18 (Pin_18)
- new net A14: J?.23 (Pin_23)
- new net A15: J?.8 (Pin_8)
- new net A3: J?.37 (Pin_37)
- new net A4: J?.39 (Pin_39)
- new net A5: J?.32 (Pin_32)
- new net A6: J?.30 (Pin_30)
- new net A7: J?.26 (Pin_26)
- new net A8: J?.28 (Pin_28)
- new net B10: J?.29 (Pin_29)
- new net B12: J?.12 (Pin_12)
- new net B14: J?.25 (Pin_25)
- new net B15: J?.21 (Pin_21)
- new net B16: J?.19 (Pin_19)
- new net B6: J?.33 (Pin_33)
- new net B8: J?.24 (Pin_24)
- new net C10: J?.10 (Pin_10)
- new net C11: J?.14 (Pin_14)
- new net C12: J?.2 (Pin_2)
- new net C14: J?.6 (Pin_6)
- new net C15: J?.15 (Pin_15)
- new net C16: J?.17 (Pin_17)
- new net C5: J?.35 (Pin_35)
- new net C6: J?.36 (Pin_36)
- new net C7: J?.34 (Pin_34)
- new net C8: J?.22 (Pin_22)
- new net C9: J?.31 (Pin_31)
- new net D5: J?.40 (Pin_40)
- new net D6: J?.38 (Pin_38)
- new net E14: J?.4 (Pin_4)
- new net E16: J?.13 (Pin_13)
- new net F16: J?.11 (Pin_11)
- new net GND: J?.1 (Pin_1), J?.27 (Pin_27), J?.27 (Pin_27), J?.9 (Pin_9), J?.9 (Pin_9)
- new net H13: J?.7 (Pin_7)
- new net J11: J?.3 (Pin_3)
- new net J13: J?.5 (Pin_5)
- new net K11: J?.2 (Pin_2)
- new net L10: J?.21 (Pin_21)
- new net L12: J?.1 (Pin_1)
- new net L13: J?.8 (Pin_8)
- new net M10: J?.25 (Pin_25)
- new net M12: J?.11 (Pin_11)
- new net M13: J?.6 (Pin_6)
- new net M4: J?.38 (Pin_38)
- new net N11: J?.19 (Pin_19)
- new net N12: J?.15 (Pin_15)
- new net N3: J?.40 (Pin_40)
- new net N4: J?.34 (Pin_34)
- new net N5: J?.35 (Pin_35)
- new net P11: J?.23 (Pin_23)
- new net P12: J?.17 (Pin_17)
- new net P2: J?.39 (Pin_39)
- new net P4: J?.36 (Pin_36)
- new net P5: J?.33 (Pin_33)
- new net P7: J?.4 (Pin_4)
- new net P8: J?.26 (Pin_26)
- new net P9: J?.22 (Pin_22)
- new net R12: J?.16 (Pin_16)
- new net R14: J?.14 (Pin_14)
- new net R15: J?.10 (Pin_10)
- new net R16: J?.13 (Pin_13)
- new net R2: J?.37 (Pin_37)
- new net R5: J?.28 (Pin_28)
- new net R7: J?.29 (Pin_29)
- new net R9: J?.24 (Pin_24)
- new net T13: J?.20 (Pin_20)
- new net T14: J?.18 (Pin_18)
- new net T15: J?.12 (Pin_12)
- new net T5: J?.32 (Pin_32)
- new net T6: J?.30 (Pin_30)
- new net T7: J?.31 (Pin_31)
- no-connect marks 0 -> 1
